File: led_controller.kicad_pcb (KiCad board)
At the start: 2 copper layers, 50 x 45 mm, 32 parts, among them IC1 ESP32-C3-MINI-1-N4X, IC2 L6983N33QTR, J1 Screw_Terminal_01x02, J2 Screw_Terminal_01x02, J3 Conn_01x04_Pin, J4 Screw_Terminal_01x02, J5 Conn_01x03_Pin, Q2 FQD13N10LTM

Commit message: Add files via upload
Parts:
- added R10: 100k, Resistor_SMD:R_0805_2012Metric_Pad1.20x1.40mm_HandSolder, F.Cu at (76.6, 37.9)
- moved R9 1.93 mm to (72.3, 37.7)
Connections:
- IC2 pad 5: 3v3 -> Net-(IC2-PGOOD)
Routing:
- net 3v3: track 158.8 -> 162.7 mm
- net Net-(IC2-PGOOD): track 0.00 -> 3.66 mm
- net Net-(IC2-FSW): track 6.20 -> 6.82 mm

Commit message: Add files via upload
Parts:
- removed L1: 4,7uH, Inductor_SMD:L_6.3x6.3_H3
- added L2: XAL6060-472MEC, desk:XAL6060472MEC, F.Cu at (84.8, 53.1)
- moved Cout1 2.43 mm to (77.4, 50.3)
Routing:
- net Net-(IC2-SW_1): track 17.2 -> 10.3 mm
- net 3v3: track 162.7 -> 165.2 mm
- net Net-(IC2-BOOT): track 7.18 -> 8.13 mm
- net GNDREF: track 14.9 -> 14.6 mm, vias 64 -> 56
- added copper zone on F.Cu, net Net-(IC2-SW_1)

Commit message: Add files via upload
Parts:
- R1, R2, R3, R4, R5, R6, R7: footprint Resistor_SMD:R_1206_3216Metric_Pad1.30x1.75mm_HandSolder -> Resistor_SMD:R_0805_2012Metric_Pad1.20x1.40mm_HandSolder
- moved R6 1.85 mm to (92.2, 56.1)
Routing:
- net Net-(J5-Pin_2): track 18.2 -> 17.4 mm
- net Net-(J5-Pin_3): track 16.5 -> 17.0 mm
- net IO7: track 7.03 -> 7.58 mm

Commit message: Add files via upload
Parts:
- R10: value 100k -> 1Mohm
- R8: value 100Ohm -> 100K
- moved Cout2 1.93 mm to (86.3, 60.5)
- turned R5 to 135 degrees
Routing:
- net VCC: track 40.5 -> 39.2 mm
- net GNDREF: track 14.6 -> 14.7 mm, vias 56 -> 88
- net (no net): vias 8 -> 0
- added copper zone on F.Cu, net VCC
