File: led_controller.kicad_pcb (KiCad board)
At the start: 2 copper layers, 50 x 45 mm, 33 parts, among them IC1 ESP32-C3-MINI-1-N4X, IC2 L6983N33QTR, J1 Screw_Terminal_01x02, J2 Screw_Terminal_01x02, J3 Conn_01x04_Pin, J4 Screw_Terminal_01x02, J5 Conn_01x03_Pin, Q2 FQD13N10LTM

Commit message: Add files via upload
Parts:
- added R11: 1k, Resistor_SMD:R_0805_2012Metric_Pad1.20x1.40mm_HandSolder, F.Cu at (93.2, 60.7)
- added status: 5973324507F, desk:5973324507F, F.Cu at (91.6, 63.3)
Connections:
- IC1 pad 6: unconnected-(IC1-IO3-Pad6) -> led
Routing:
- net led: track 0.00 -> 23.2 mm, vias 0 -> 2
- net Net-(LED1-K): track 0.00 -> 2.68 mm

Commit message: Add files via upload
Parts:
- removed Q2: FQD13N10LTM, desk:FDD4685F085
- removed status: 5973324507F, desk:5973324507F
- added LED1: 5973324507F, desk:5973324507F, F.Cu at (91.6, 63.1)
- added Q1: STD120N4LF6, desk:STD120N4LF6, B.Cu at (95.7, 40.1)
Routing:
- net DIM-: track 7.18 -> 8.31 mm
- net Net-(Q1-G): track 9.52 -> 8.58 mm
Other:
- board text added: "status"
