File: led_controller.kicad_sch (KiCad schematic)
At the start: 32 parts, among them IC1 ESP32-C3-MINI-1-N4X, IC2 L6983N33QTR, J1 Screw_Terminal_01x02, J2 Screw_Terminal_01x02, J3 Conn_01x04_Pin, J4 Screw_Terminal_01x02, J5 Conn_01x03_Pin, Q2 FQD13N10LTM

Commit message: Add files via upload
Parts:
- added R10: 100k, Resistor_SMD:R_0805_2012Metric_Pad1.20x1.40mm_HandSolder, symbol Device:R
Connections:
- net 3v3: now also R10.1; no longer IC2.5 (PGOOD)
- new net: IC2.5 (PGOOD), R10.2
Changed lines of the file:
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@@
 	)
 	(junction
-		(at 128.27 39.37)
-		(diameter 0)
-		(color 0 0 0 0)
-	)
-	(junction
 		(at 116.84 39.37)
 		(diameter 0)
@@
 	(wire
 		(pts
-			(xy 39.37 40.64) (xy 46.99 40.64)
+			(xy 39.37 43.18) (xy 44.45 43.18)
 		)
 		(stroke
@@
 	(wire
 		(pts
-			(xy 125.73 39.37) (xy 128.27 39.37)
+			(xy 125.73 39.37) (xy 129.54 39.37)
 		)
 		(stroke
@@
 	(wire
 		(pts
-			(xy 148.59 138.43) (xy 148.59 140.97)
+			(xy 46.99 36.83) (xy 46.99 31.75)
 		)
 		(stroke
@@
 	(wire
 		(pts
-			(xy 115.57 120.65) (xy 81.28 120.65)
+			(xy 148.59 138.43) (xy 148.59 140.97)
 		)
 		(stroke
@@
 	(wire
 		(pts
-			(xy 148.59 110.49) (xy 148.59 113.03)
+			(xy 115.57 120.65) (xy 81.28 120.65)
 		)
 		(stroke
@@
 	(wire
 		(pts
-			(xy 138.43 34.29) (xy 138.43 39.37)
+			(xy 148.59 110.49) (xy 148.59 113.03)
 		)
 		(stroke
@@
 	(wire
 		(pts
-			(xy 43.18 54.61) (xy 43.18 50.8)
+			(xy 138.43 34.29) (xy 138.43 39.37)
 		)
 		(stroke
@@
 	(wire
 		(pts
-			(xy 36.83 137.16) (xy 57.15 137.16)
+			(xy 43.18 54.61) (xy 43.18 50.8)
 		)
 		(stroke
@@
 	(wire
 		(pts
-			(xy 184.15 59.69) (xy 189.23 59.69)
+			(xy 36.83 137.16) (xy 57.15 137.16)
 		)
 		(stroke
@@
 	(wire
 		(pts
-			(xy 128.27 39.37) (xy 129.54 39.37)
+			(xy 184.15 59.69) (xy 189.23 59.69)
 		)
 		(stroke
@@
 	(wire
 		(pts
-			(xy 209.55 128.27) (xy 209.55 137.16)
+			(xy 44.45 36.83) (xy 46.99 36.83)
 		)
 		(stroke
@@
 	(wire
 		(pts
-			(xy 104.14 100.33) (xy 115.57 100.33)
+			(xy 209.55 128.27) (xy 209.55 137.16)
 		)
 		(stroke
@@
 	(wire
 		(pts
-			(xy 109.22 31.75) (xy 116.84 31.75)
+			(xy 104.14 100.33) (xy 115.57 100.33)
 		)
 		(stroke
@@
 	(wire
 		(pts
-			(xy 128.27 29.21) (xy 128.27 39.37)
+			(xy 109.22 31.75) (xy 116.84 31.75)
 		)
 		(stroke
@@
 	(wire
 		(pts
-			(xy 39.37 43.18) (xy 39.37 40.64)
-		)
-		(stroke
-			(width 0)
-			(type default)
-		)
-	)
-	(wire
-		(pts
 			(xy 205.74 118.11) (xy 205.74 119.38)
 		)
@@
 	(wire
 		(pts
-			(xy 46.99 31.75) (xy 46.99 40.64)
+			(xy 44.45 36.83) (xy 44.45 43.18)
 		)
 		(stroke
@@
 		)
 	)
-	(global_label "VCC"
+	(global_label "3v3"
 		(shape input)
-		(at 189.23 57.15 90)
+		(at 52.07 39.37 180)
 		(fields_autoplaced yes)
 		(effects
@@
 				(size 1.27 1.27)
 			)
-			(justify left)
+			(justify right)
 		)
 		(property "Intersheetrefs" "${INTERSHEET_REFS}"
-			(at 189.23 50.5362 90)
+			(at 45.6982 39.37 0)
 			(effects
 				(font
 					(size 1.27 1.27)
 				)
-				(justify left)
+				(justify right)
 				(hide yes)
 			)
 		)
 	)
-	(global_label "3v3"
+	(global_label "VCC"
 		(shape input)
-		(at 27.94 143.51 180)
+		(at 189.23 57.15 90)
 		(fields_autoplaced yes)
 		(effects
@@
 				(size 1.27 1.27)
 			)
-			(justify right)
+			(justify left)
 		)
 		(property "Intersheetrefs" "${INTERSHEET_REFS}"
-			(at 21.5682 143.51 0)
+			(at 189.23 50.5362 90)
 			(effects
 				(font
 					(size 1.27 1.27)
 				)
-				(justify right)
+				(justify left)
 				(hide yes)
 			)
 		)
 	)
-	(global_label "To3v3"
+	(global_label "3v3"
 		(shape input)
-		(at 128.27 29.21 90)
+		(at 27.94 143.51 180)
 		(fields_autoplaced yes)
 		(effects
@@
 				(size 1.27 1.27)
 			)
-			(justify left)
+			(justify right)
 		)
 		(property "Intersheetrefs" "${INTERSHEET_REFS}"
-			(at 128.27 20.7216 90)
+			(at 21.5682 143.51 0)
 			(effects
 				(font
 					(size 1.27 1.27)
 				)
-				(justify left)
+				(justify right)
 				(hide yes)
 			)
@@
 		)
 	)
-	(global_label "To3v3"
-		(shape input)
-		(at 59.69 39.37 180)
-		(fields_autoplaced yes)
-		(effects
-			(font
-				(size 1.27 1.27)
-			)
-			(justify right)
-		)
-		(property "Intersheetrefs" "${INTERSHEET_REFS}"
-			(at 51.2016 39.37 0)
-			(effects
-				(font
-					(size 1.27 1.27)
-				)
-				(justify right)
-				(hide yes)
-			)
-		)
-	)
 	(global_label "IO5"
 		(shape input)
@@
 					(unit 1)
 				)
+			)
+		)
+	)
+	(symbol
+		(lib_id "Device:R")
+		(at 55.88 39.37 90)
+		(unit 1)
+		(exclude_from_sim no)
+		(in_bom yes)
+		(on_board yes)
+		(dnp no)
+		(property "Reference" "R10"
+			(at 55.626 39.624 90)
+			(effects
+				(font
+					(size 1.27 1.27)
+				)
+			)
+		)
+		(property "Value" "100k"
+			(at 55.88 38.354 90)
+			(effects
+				(font
+					(size 1.27 1.27)
+				)
+			)
+		)
+		(property "Footprint" "Resistor_SMD:R_0805_2012Metric_Pad1.20x1.40mm_HandSolder"
+			(at 55.88 41.148 90)
+			(effects
+				(font
+					(size 1.27 1.27)
+				)
+				(hide yes)
+			)
+		)
+		(property "Datasheet" "~"
+			(at 55.88 39.37 0)
+			(effects
+				(font
+					(size 1.27 1.27)
+				)
+				(hide yes)
+			)
+		)
+		(property "Description" "Resistor"
+			(at 55.88 39.37 0)
+			(effects
+				(font
+					(size 1.27 1.27)
+				)
+				(hide yes)
+			)
+		)
+		(pin "1"
+		)
+		(pin "2"
+		)
+		(instances
+			(project "led_controller"
+				(path "/f7384fac-022b-47e0-8e4e-5c549011b8cf"
+					(reference "R10")
+					(unit 1)
+				)

Commit message: Add files via upload
Parts:
- removed L1: 4,7uH, Inductor_SMD:L_6.3x6.3_H3, symbol Device:L
- added L2: XAL6060-472MEC, desk:XAL6060472MEC, symbol desk:XAL6060-472MEC
Connections:
- net 3v3: now also L2.2
- net at Cout1.2, IC2.14 (SW_1), IC2.15 (SW_2): now also L2.1
Other:
- moved on the sheet: Cout2
Changed lines of the file:
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@@
 	)
 	(junction
-		(at 129.54 39.37)
+		(at 142.24 39.37)
 		(diameter 0)
 		(color 0 0 0 0)
@@
 	)
 	(junction
-		(at 138.43 39.37)
+		(at 151.13 39.37)
 		(diameter 0)
 		(color 0 0 0 0)
 	)
 	(junction
-		(at 125.73 39.37)
+		(at 138.43 39.37)
 		(diameter 0)
 		(color 0 0 0 0)
@@
 	(wire
 		(pts
-			(xy 125.73 29.21) (xy 125.73 39.37)
+			(xy 138.43 29.21) (xy 138.43 39.37)
 		)
 		(stroke
@@
 	(wire
 		(pts
-			(xy 129.54 40.64) (xy 129.54 39.37)
+			(xy 142.24 40.64) (xy 142.24 39.37)
 		)
 		(stroke
@@
 	(wire
 		(pts
-			(xy 129.54 39.37) (xy 138.43 39.37)
+			(xy 142.24 39.37) (xy 151.13 39.37)
 		)
 		(stroke
@@
 	(wire
 		(pts
-			(xy 125.73 39.37) (xy 129.54 39.37)
+			(xy 138.43 39.37) (xy 142.24 39.37)
 		)
 		(stroke
@@
 	(wire
 		(pts
-			(xy 124.46 39.37) (xy 125.73 39.37)
+			(xy 137.16 39.37) (xy 138.43 39.37)
 		)
 		(stroke
@@
 	(wire
 		(pts
-			(xy 138.43 34.29) (xy 138.43 39.37)
+			(xy 151.13 34.29) (xy 151.13 39.37)
 		)
 		(stroke
@@
 	(wire
 		(pts
-			(xy 138.43 39.37) (xy 139.7 39.37)
+			(xy 151.13 39.37) (xy 152.4 39.37)
 		)
 		(stroke
@@
 	(wire
 		(pts
-			(xy 129.54 48.26) (xy 129.54 52.07)
+			(xy 142.24 48.26) (xy 142.24 52.07)
 		)
 		(stroke
@@
 	(global_label "Vbias"
 		(shape input)
-		(at 125.73 29.21 90)
+		(at 138.43 29.21 90)
 		(fields_autoplaced yes)
 		(effects
@@
 		)
 		(property "Intersheetrefs" "${INTERSHEET_REFS}"
-			(at 125.73 21.2053 90)
+			(at 138.43 21.2053 90)
 			(effects
 				(font
@@
 	(global_label "FbOut"
 		(shape input)
-		(at 138.43 34.29 90)
+		(at 151.13 34.29 90)
 		(fields_autoplaced yes)
 		(effects
@@
 		)
 		(property "Intersheetrefs" "${INTERSHEET_REFS}"
-			(at 138.43 25.862 90)
+			(at 151.13 25.862 90)
 			(effects
 				(font
@@
 	(global_label "3v3"
 		(shape input)
-		(at 139.7 39.37 0)
+		(at 152.4 39.37 0)
 		(fields_autoplaced yes)
 		(effects
@@
 		)
 		(property "Intersheetrefs" "${INTERSHEET_REFS}"
-			(at 146.0718 39.37 0)
+			(at 158.7718 39.37 0)
 			(effects
 				(font
@@
 	)
 	(symbol
-		(lib_id "Device:L")
-		(at 120.65 39.37 90)
-		(unit 1)
-		(exclude_from_sim no)
-		(in_bom yes)
-		(on_board yes)
-		(dnp no)
-		(fields_autoplaced yes)
-		(property "Reference" "L1"
-			(at 120.65 34.29 90)
-			(effects
-				(font
-					(size 1.27 1.27)
-				)
-				(hide yes)
-			)
-		)
-		(property "Value" "4,7uH"
-			(at 120.65 36.83 90)
-			(effects
-				(font
-					(size 1.27 1.27)
-				)
-			)
-		)
-		(property "Footprint" "Inductor_SMD:L_6.3x6.3_H3"
-			(at 120.65 39.37 0)
-			(effects
-				(font
-					(size 1.27 1.27)
-				)
-				(hide yes)
-			)
-		)
-		(property "Datasheet" "~"
-			(at 120.65 39.37 0)
-			(effects
-				(font
-					(size 1.27 1.27)
-				)
-				(hide yes)
-			)
-		)
-		(property "Description" "Inductor"
-			(at 120.65 39.37 0)
-			(effects
-				(font
-					(size 1.27 1.27)
-				)
-				(hide yes)
-			)
-		)
-		(pin "1"
-		)
-		(pin "2"
-		)
-		(instances
-			(project ""
-				(path "/f7384fac-022b-47e0-8e4e-5c549011b8cf"
-					(reference "L1")
-					(unit 1)
-				)
-			)
-		)
-	)
-	(symbol
 		(lib_id "Device:R")
 		(at 43.18 31.75 90)
@@
 	(symbol
 		(lib_id "power:GNDREF")
-		(at 129.54 52.07 0)
+		(at 142.24 52.07 0)
 		(unit 1)
 		(exclude_from_sim no)
@@
 		(fields_autoplaced yes)
 		(property "Reference" "#PWR04"
-			(at 129.54 58.42 0)
+			(at 142.24 58.42 0)
 			(effects
 				(font
@@
 		)
 		(property "Value" "GNDREF"
-			(at 129.54 57.15 0)
+			(at 142.24 57.15 0)
 			(effects
 				(font
@@
 		)
 		(property "Footprint" ""
-			(at 129.54 52.07 0)
+			(at 142.24 52.07 0)
 			(effects
 				(font
@@
 		)
 		(property "Datasheet" ""
-			(at 129.54 52.07 0)
+			(at 142.24 52.07 0)
 			(effects
 				(font
@@
 		)
 		(property "Description" "Power symbol creates a global label with name \"GNDREF\" , reference supply ground"
-			(at 129.54 52.07 0)
+			(at 142.24 52.07 0)
 			(effects
 				(font
@@
 	)
 	(symbol
+		(lib_id "desk:XAL6060-472MEC")
+		(at 116.84 39.37 0)
+		(unit 1)
+		(exclude_from_sim no)
+		(in_bom yes)
+		(on_board yes)
+		(dnp no)
+		(fields_autoplaced yes)
+		(property "Reference" "L2"
+			(at 127 33.02 0)
+			(effects
+				(font
+					(size 1.27 1.27)
+				)
+			)
+		)
+		(property "Value" "XAL6060-472MEC"
+			(at 127 35.56 0)
+			(effects
+				(font
+					(size 1.27 1.27)
+				)
+			)
+		)
+		(property "Footprint" "desk:XAL6060472MEC"
+			(at 133.35 135.56 0)
+			(effects
+				(font
+					(size 1.27 1.27)
+				)
+				(justify left top)
+				(hide yes)
+			)
+		)
+		(property "Datasheet" "https://componentsearchengine.com/Datasheets/2/XAL6060-472MEC.pdf"
+			(at 133.35 235.56 0)
+			(effects
+				(font
+					(size 1.27 1.27)
+				)
+				(justify left top)
+				(hide yes)
+			)
+		)
+		(property "Description" "Fixed Inductors 4.7uH 20% 11A 14.40mOhms AEC-Q200"
+			(at 116.84 39.37 0)
+			(effects
+				(font
+					(size 1.27 1.27)
+				)
+				(hide yes)
+			)
+		)
+		(property "Height" "6.1"
+			(at 133.35 435.56 0)
+			(effects
+				(font
+					(size 1.27 1.27)
+				)
+				(justify left top)
+				(hide yes)
+			)
+		)
+		(property "Manufacturer_Name" "COILCRAFT"
+			(at 133.35 535.56 0)
+			(effects
+				(font
+					(size 1.27 1.27)
+				)
+				(justify left top)
+				(hide yes)
+			)
+		)
+		(property "Manufacturer_Part_Number" "XAL6060-472MEC"
+			(at 133.35 635.56 0)
+			(effects
+				(font
+					(size 1.27 1.27)
+				)
+				(justify left top)
+				(hide yes)
+			)
+		)
+		(property "Mouser Part Number" "994-XAL6060-472MEC"
+			(at 133.35 735.56 0)
+			(effects
+				(font
+					(size 1.27 1.27)
+				)
+				(justify left top)
+				(hide yes)
+			)
+		)
+		(property "Mouser Price/Stock" "https://www.mouser.co.uk/ProductDetail/Coilcraft/XAL6060-472MEC?qs=zCSbvcPd3pajUkm1Owi1LA%3D%3D"
+			(at 133.35 835.56 0)
+			(effects
+				(font
+					(size 1.27 1.27)
+				)
+				(justify left top)
+				(hide yes)
+			)
+		)
+		(property "Arrow Part Number" ""
+			(at 133.35 935.56 0)
+			(effects
+				(font
+					(size 1.27 1.27)
+				)
+				(justify left top)
+				(hide yes)
+			)
+		)
+		(property "Arrow Price/Stock" ""
+			(at 133.35 1035.56 0)
+			(effects
+				(font
+					(size 1.27 1.27)
+				)
+				(justify left top)
+				(hide yes)
+			)
+		)
+		(pin "1"
+		)
+		(pin "2"
+		)
+		(instances
+			(project ""
+				(path "/f7384fac-022b-47e0-8e4e-5c549011b8cf"
+					(reference "L2")
+					(unit 1)
+				)
+			)
+		)
+	)
+	(symbol
 		(lib_id "power:GNDREF")
 		(at 205.74 119.38 0)
@@
 	(symbol
 		(lib_id "Device:C")
-		(at 129.54 44.45 0)
+		(at 142.24 44.45 0)
 		(unit 1)
 		(exclude_from_sim no)
@@
 		(fields_autoplaced yes)
 		(property "Reference" "Cout2"
-			(at 133.35 43.1799 0)
+			(at 146.05 43.1799 0)
 			(effects
 				(font
@@
 		)
 		(property "Value" "47uF"
-			(at 133.35 45.7199 0)
+			(at 146.05 45.7199 0)
 			(effects
 				(font
@@
 		)
 		(property "Footprint" "Capacitor_SMD:C_1206_3216Metric_Pad1.33x1.80mm_HandSolder"
-			(at 130.5052 48.26 0)
+			(at 143.2052 48.26 0)
 			(effects
 				(font
@@
 		)
 		(property "Datasheet" "~"
-			(at 129.54 44.45 0)
+			(at 142.24 44.45 0)
 			(effects
 				(font
@@
 		)
 		(property "Description" "Unpolarized capacitor"
-			(at 129.54 44.45 0)
+			(at 142.24 44.45 0)
 			(effects
 				(font

Commit message: Add files via upload
Parts:
- R1, R2, R3, R4, R5, R6, R7: footprint Resistor_SMD:R_1206_3216Metric_Pad1.30x1.75mm_HandSolder -> Resistor_SMD:R_0805_2012Metric_Pad1.20x1.40mm_HandSolder
Changed lines of the file:
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@@
 			)
 		)
-		(property "Footprint" "Resistor_SMD:R_1206_3216Metric_Pad1.30x1.75mm_HandSolder"
+		(property "Footprint" "Resistor_SMD:R_0805_2012Metric_Pad1.20x1.40mm_HandSolder"
 			(at 33.02 118.618 90)
 			(effects
@@
 			)
 		)
-		(property "Footprint" "Resistor_SMD:R_1206_3216Metric_Pad1.30x1.75mm_HandSolder"
+		(property "Footprint" "Resistor_SMD:R_0805_2012Metric_Pad1.20x1.40mm_HandSolder"
 			(at 186.69 149.098 90)
 			(effects
@@
 			)
 		)
-		(property "Footprint" "Resistor_SMD:R_1206_3216Metric_Pad1.30x1.75mm_HandSolder"
+		(property "Footprint" "Resistor_SMD:R_0805_2012Metric_Pad1.20x1.40mm_HandSolder"
 			(at 31.75 145.288 90)
 			(effects
@@
 			)
 		)
-		(property "Footprint" "Resistor_SMD:R_1206_3216Metric_Pad1.30x1.75mm_HandSolder"
+		(property "Footprint" "Resistor_SMD:R_0805_2012Metric_Pad1.20x1.40mm_HandSolder"
 			(at 197.358 91.44 90)
 			(effects
@@
 			)
 		)
-		(property "Footprint" "Resistor_SMD:R_1206_3216Metric_Pad1.30x1.75mm_HandSolder"
+		(property "Footprint" "Resistor_SMD:R_0805_2012Metric_Pad1.20x1.40mm_HandSolder"
 			(at 191.77 89.408 90)
 			(effects
@@
 			)
 		)
-		(property "Footprint" "Resistor_SMD:R_1206_3216Metric_Pad1.30x1.75mm_HandSolder"
+		(property "Footprint" "Resistor_SMD:R_0805_2012Metric_Pad1.20x1.40mm_HandSolder"
 			(at 180.34 61.468 90)
 			(effects
@@
 			)
 		)
-		(property "Footprint" "Resistor_SMD:R_1206_3216Metric_Pad1.30x1.75mm_HandSolder"
+		(property "Footprint" "Resistor_SMD:R_0805_2012Metric_Pad1.20x1.40mm_HandSolder"
 			(at 186.69 138.938 90)
 			(effects

Commit message: Add files via upload
Parts:
- R10: value 100k -> 1Mohm
- R8: value 100Ohm -> 100K
Changed lines of the file:
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@@
 			)
 		)
-		(property "Value" "100Ohm"
+		(property "Value" "100K"
 			(at 43.18 27.94 90)
 			(effects
@@
 			)
 		)
-		(property "Value" "100k"
+		(property "Value" "1Mohm"
 			(at 55.88 38.354 90)
 			(effects

Commit message: Add files via upload
Parts:
- added LED1: 5973324507F, desk:5973324507F, symbol desk:5973324507F
- added R11: 1k, Resistor_SMD:R_0805_2012Metric_Pad1.20x1.40mm_HandSolder, symbol Device:R
Connections:
- net GNDREF: now also LED1.2 (A)
- net led: now reaches IC1.6 (IO3)
- net led: now also R11.1
- new net: LED1.1 (K), R11.2
- no-connect marks 22 -> 21

Commit message: Add files via upload
Parts:
- removed Q2: FQD13N10LTM, desk:FDD4685F085, symbol desk:FQD13N10LTM
- added Q1: STD120N4LF6, desk:STD120N4LF6, symbol desk:STD120N4LF6
Connections:
- net DIM-: now also Q1.2 (D)
- net GNDREF: now also Q1.3 (S)
- net at R1.2, R4.2: now also Q1.1 (G)
Changed lines of the file:
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@@
-	)
-	(symbol
-		(lib_id "desk:FQD13N10LTM")
-		(at 199.39 87.63 0)
-		(unit 1)
-		(exclude_from_sim no)
-		(in_bom yes)
-		(on_board yes)
-		(dnp no)
-		(fields_autoplaced yes)
-		(property "Reference" "Q2"
-			(at 210.82 83.8199 0)
-			(effects
-				(font
-					(size 1.27 1.27)
-				)
-				(justify left)
-			)
-		)
-		(property "Value" "FQD13N10LTM"
-			(at 210.82 86.3599 0)
-			(effects
-				(font
-					(size 1.27 1.27)
-				)
-				(justify left)
-			)
-		)
-		(property "Footprint" "desk:FDD4685F085"
-			(at 210.82 186.36 0)
-			(effects
-				(font
-					(size 1.27 1.27)
-				)
-				(justify left top)
-				(hide yes)
-			)
-		)
-		(property "Datasheet" "https://www.onsemi.com/pub/Collateral/FQU13N10L-D.pdf"
-			(at 210.82 286.36 0)
-			(effects
-				(font
-					(size 1.27 1.27)
-				)
-				(justify left top)
-				(hide yes)
-			)
-		)
-		(property "Description" "10A, 100V, RDS(on) = 180m(Max.) @VGS = 10 V, ID = 5A; 100% avalanche tested; Low Crss ( Typ. 20pF); Low gate charge ( Typ. 8.7nC)"
-			(at 199.39 87.63 0)
-			(effects
-				(font
-					(size 1.27 1.27)
-				)
-				(hide yes)
-			)
-		)
-		(property "Height" ""
-			(at 210.82 486.36 0)
-			(effects
-				(font
-					(size 1.27 1.27)
-				)
-				(justify left top)
-				(hide yes)
-			)
-		)
-		(property "Manufacturer_Name" "onsemi"
-			(at 210.82 586.36 0)
-			(effects
-				(font
-					(size 1.27 1.27)
-				)
-				(justify left top)
-				(hide yes)
-			)
-		)
-		(property "Manufacturer_Part_Number" "FQD13N10LTM"
-			(at 210.82 686.36 0)
-			(effects
-				(font
-					(size 1.27 1.27)
-				)
-				(justify left top)
-				(hide yes)
-			)
-		)
-		(property "Mouser Part Number" "512-FQD13N10LTM"
-			(at 210.82 786.36 0)
-			(effects
-				(font
-					(size 1.27 1.27)
-				)
-				(justify left top)
-				(hide yes)
-			)
-		)
-		(property "Mouser Price/Stock" "https://www.mouser.co.uk/ProductDetail/onsemi-Fairchild/FQD13N10LTM?qs=q8yi3gPquyEw5NK8D9%252Bd2A%3D%3D"
-			(at 210.82 886.36 0)
-			(effects
-				(font
-					(size 1.27 1.27)
-				)
-				(justify left top)
-				(hide yes)
-			)
-		)
-		(property "Arrow Part Number" "FQD13N10LTM"
-			(at 210.82 986.36 0)
-			(effects
-				(font
-					(size 1.27 1.27)
-				)
-				(justify left top)
-				(hide yes)
-			)
-		)
-		(property "Arrow Price/Stock" "https://www.arrow.com/en/products/fqd13n10ltm/on-semiconductor?utm_currency=USD&region=nac"
-			(at 210.82 1086.36 0)
-			(effects
-				(font
-					(size 1.27 1.27)
-				)
-				(justify left top)
-				(hide yes)
-			)
-		)
-		(pin "3"
-		)
-		(pin "2"
-		)
-		(pin "1"
-		)
-		(instances
-			(project ""
-				(path "/f7384fac-022b-47e0-8e4e-5c549011b8cf"
-					(reference "Q2")
-					(unit 1)
-				)
-			)
-		)
 	)
 	(symbol
@@
 					(unit 1)
 				)
+			)
+		)
+	)
+	(symbol
+		(lib_id "desk:STD120N4LF6")
+		(at 199.39 87.63 0)
+		(unit 1)
+		(exclude_from_sim no)
+		(in_bom yes)
+		(on_board yes)
+		(dnp no)
+		(fields_autoplaced yes)
+		(property "Reference" "Q1"
+			(at 210.82 83.8199 0)
+			(effects
+				(font
+					(size 1.27 1.27)
+				)
+				(justify left)
+			)
+		)
+		(property "Value" "STD120N4LF6"
+			(at 210.82 86.3599 0)
+			(effects
+				(font
+					(size 1.27 1.27)
+				)
+				(justify left)
+			)
+		)
+		(property "Footprint" "desk:STD120N4LF6"
+			(at 210.82 87.6299 0)
+			(effects
+				(font
+					(size 1.27 1.27)
+				)
+				(justify left)
+				(hide yes)
+			)
+		)
+		(property "Datasheet" "https://www.st.com/resource/en/datasheet/stb120n4lf6.pdf"
+			(at 210.82 286.36 0)
+			(effects
+				(font
+					(size 1.27 1.27)
+				)
+				(justify left top)
+				(hide yes)
+			)
+		)
+		(property "Description" "N-Channel 40 V 80A (Tc) 110W (Tc) Surface Mount DPAK , 4mOhm @ 40A, 10V , 4300 pF @ 25V , 110W (Tc) , -55C ~ 175C (TJ)"
+			(at 199.39 87.63 0)
+			(effects
+				(font
+					(size 1.27 1.27)
+				)
+				(hide yes)
+			)
+		)
+		(property "Height" "2.4"
+			(at 210.82 486.36 0)
+			(effects
+				(font
+					(size 1.27 1.27)
+				)
+				(justify left top)
+				(hide yes)
+			)
+		)
+		(property "Manufacturer_Name" "STMicroelectronics"
+			(at 210.82 586.36 0)
+			(effects
+				(font
+					(size 1.27 1.27)
+				)
+				(justify left top)
+				(hide yes)
+			)
+		)
+		(property "Manufacturer_Part_Number" "STD120N4LF6"
+			(at 210.82 686.36 0)
+			(effects
+				(font
+					(size 1.27 1.27)
+				)
+				(justify left top)
+				(hide yes)
+			)
+		)
+		(property "Mouser Part Number" "511-STD120N4LF6"
+			(at 210.82 786.36 0)
+			(effects
+				(font
+					(size 1.27 1.27)
+				)
+				(justify left top)
+				(hide yes)
+			)
+		)
+		(property "Mouser Price/Stock" "https://www.mouser.co.uk/ProductDetail/STMicroelectronics/STD120N4LF6?qs=CBOTe0%252BbgkZMffiWp8DgqQ%3D%3D"
+			(at 210.82 886.36 0)
+			(effects
+				(font
+					(size 1.27 1.27)
+				)
+				(justify left top)
+				(hide yes)
+			)
+		)
+		(property "Arrow Part Number" "STD120N4LF6"
+			(at 210.82 986.36 0)
+			(effects
+				(font
+					(size 1.27 1.27)
+				)
+				(justify left top)
+				(hide yes)
+			)
+		)
+		(property "Arrow Price/Stock" "https://www.arrow.com/en/products/std120n4lf6/stmicroelectronics?utm_currency=USD&region=nac"
+			(at 210.82 1086.36 0)
+			(effects
+				(font
+					(size 1.27 1.27)
+				)
+				(justify left top)
+				(hide yes)
+			)
+		)
+		(pin "1"
+		)
+		(pin "2"
+		)
+		(pin "3"
+		)
+		(instances
+			(project ""
+				(path "/f7384fac-022b-47e0-8e4e-5c549011b8cf"
+					(reference "Q1")
+					(unit 1)
+				)
